File: hardware/usb2can.sch (EAGLE design)
At the start: 43 parts, among them IC1 7805TV, U1 ATMEGA32U4, U2 MCP2551SN, U3 MCP2510SO, X2 USB-A-S

Commit message: added the CAN Start of Frame signal path to pcb
Connections:
- new net CAN_SOF: U1PORTB.(OC1B/PCINT6/OC4B/ADC13)PB6, U3>NAME.CLKOUT
Changed lines of the file:
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@@
+</segment>
+</net>
+<net name="CAN_SOF" class="0">
+<segment>
+<pinref part="U3" gate="&gt;NAME" pin="CLKOUT"/>
+<wire x1="149.86" y1="25.4" x2="162.56" y2="25.4" width="0.1524" layer="91"/>
+<label x="154.94" y="25.4" size="1.778" layer="95"/>
+</segment>
+<segment>
+<pinref part="U1" gate="PORTB" pin="(OC1B/PCINT6/OC4B/ADC13)PB6"/>
+<wire x1="60.96" y1="60.96" x2="73.66" y2="60.96" width="0.1524" layer="91"/>
+<label x="68.58" y="60.96" size="1.778" layer="95"/>
 </segment>
 </net>
